Commit message: добавил изменения

File: src/mobile_description/urdf/robot_v1.urdf (robot description, URDF)
Before this commit: robot vehicle_blue, 5 links, 4 joints
Links:
- added link vehicle_blue/chassis/gpu_lidar; visual cylinder length=0.1 radius=0.1
Joints:
- added joint lidar_joint: type fixed, parent chassis, child vehicle_blue/chassis/gpu_lidar, origin xyz=0.8 0 0.35 rpy=0 0 0
- joint camera_joint: origin xyz=1.0 0 0.25 rpy=0 0 1.5708 -> xyz=1.0 0 0.25 rpy=0 0 0

Commit message: переименовал test_world.sdf в world_v1.sdf

File: src/mobile_description/urdf/robot_v1.urdf (robot description, URDF)
Before this commit: robot vehicle_blue, 6 links, 5 joints
Joints:
- joint lidar_joint: origin xyz=0.8 0 0.35 rpy=0 0 0 -> xyz=0.8 0 0.3 rpy=0 0 0
